Commit message: feat(gazebo): finalize industrial agentic acceptance

File: extensions/gazebo/assets/rm75_6fb_v_vendor/urdf/arm_ros2_control.xacro (robot description, xacro)
@@ -2,8 +2,8 @@
 <robot xmlns:xacro="http://www.ros.org/wiki/xacro">
   <xacro:macro name="rm75_v_arm_control_interfaces">
-    <xacro:macro name="rm75_v_arm_interface" params="name">
+    <xacro:macro name="rm75_v_arm_interface" params="name initial_value:=0.0">
       <joint name="${name}">
         <command_interface name="position"/>
-        <state_interface name="position"><param name="initial_value">0.0</param></state_interface>
+        <state_interface name="position"><param name="initial_value">${initial_value}</param></state_interface>
         <state_interface name="velocity"/>
       </joint>
@@ -15,5 +15,7 @@
     <xacro:rm75_v_arm_interface name="joint_5"/>
     <xacro:rm75_v_arm_interface name="joint_6"/>
-    <xacro:rm75_v_arm_interface name="joint_7"/>
+    <!-- Keep the terminal wrist square with the 180-degree pedestal
+         installation so the gripper and rear camera share a workcell axis. -->
+    <xacro:rm75_v_arm_interface name="joint_7" initial_value="3.141592653589793"/>
   </xacro:macro>
 </robot>

File: extensions/gazebo/assets/rm75_6fb_v_vendor/urdf/rm75_6fb_v.urdf.xacro (robot description, xacro)
@@ -88,7 +88,11 @@
     name="joint_1"
     type="revolute">
+    <!-- Workcell mounting transform: the RM75 pedestal faces away from the
+         work table.  Keep this rotation inside the kinematic tree (rather
+         than applying a Gazebo-only spawn yaw) so TF, MoveIt, IK, collision
+         checking, and the rendered robot all share the same base frame. -->
     <origin
       xyz="0 0 0.2405"
-      rpy="0 0 0" />
+      rpy="0 0 3.14159265359" />
     <parent
       link="base_link" />
@@ -451,113 +455,122 @@
       velocity="3.14" />
   </joint>
-  <link
-    name="camera_rolink">
-    <inertial>
-      <origin
-        xyz="0.0080749 -0.044495 0.0085055"
-        rpy="0 0 0" />
-      <mass
-        value="0.019695" />
-      <inertia
-        ixx="1.5115E-05"
-        ixy="-1.9139E-06"
-        ixz="-8.811E-09"
-        iyy="2.7638E-06"
-        iyz="6.7136E-09"
-        izz="1.399E-05" />
-    </inertial>
-    <visual>
-      <origin
-        xyz="0 0 0"
-        rpy="0 0 0" />
-      <geometry>
-        <mesh
-          filename="package://openeta_rm75_v_description/meshes/camera_rolink.STL" />
-      </geometry>
-      <material
-        name="">
-        <color
-          rgba="0.75294 0.75294 0.75294 1" />
-      </material>
-    </visual>
-    <collision>
-      <origin
-        xyz="0 0 0"
-        rpy="0 0 0" />
-      <geometry>
-        <mesh
-          filename="package://openeta_rm75_v_description/meshes/camera_rolink.STL" />
-      </geometry>
-    </collision>
-  </link>
-  <joint
-    name="camera_rojoint"
-    type="fixed">
-    <origin
-      xyz="-0.033 -0.0085 -0.05388"
-      rpy="1.5708 -1.5708 3.1416" />
-    <parent
-      link="link_7" />
-    <child
-      link="camera_rolink" />
-  </joint>
-  <link
-    name="camera_link">
-    <inertial>
-      <origin
-        xyz="-0.009 -1.1052E-09 -0.011436"
-        rpy="0 0 0" />
-      <mass
-        value="0.03915" />
-      <inertia
-        ixx="7.2029E-06"
-        ixy="1.2847E-13"
-        ixz="4.6827E-14"
-        iyy="7.199E-06"
-        iyz="4.4495E-13"
-        izz="1.1014E-05" />
-    </inertial>
-    <visual>
-      <origin
-        xyz="0 0 0"
-        rpy="0 0 0" />
-      <geometry>
-        <mesh
-          filename="package://openeta_rm75_v_description/meshes/camera_link.STL" />
-      </geometry>
-      <material
-        name="">
-        <color
-          rgba="0.79216 0.81961 0.93333 1" />
-      </material>
-    </visual>
-    <collision>
-      <origin
-        xyz="0 0 0"
-        rpy="0 0 0" />
-      <geometry>
-        <mesh
-          filename="package://openeta_rm75_v_description/meshes/camera_link.STL" />
-      </geometry>
-    </collision>
-  </link>
-  <joint
-    name="camera_joint"
-    type="fixed">
-    <origin
-      xyz="0.029031 -0.10022 -0.0005"
-      rpy="0 1.5708 0" />
-    <parent
-      link="camera_rolink" />
-    <child
-      link="camera_link" />
+  <!-- Keep the manufacturer's physical wrist-camera mounting datum and mesh.
+       The full-length arm is pitched toward the tool tip below.  This keeps
+       the optical ray clear of the wrist and gripper body; shortening this
+       arm makes their fixed self-occlusion dominate every eye-in-hand view. -->
+  <link name="wrist_camera_bracket_link">
+    <inertial>
+      <origin xyz="0.0080749 -0.0222475 0.0085055" rpy="0 0 0" />
+      <mass value="0.010" />
+      <inertia ixx="4.0E-06" ixy="-5.0E-07" ixz="0"
+               iyy="1.4E-06" iyz="0" izz="3.8E-06" />
+    </inertial>
+    <visual name="wrist_camera_vendor_bracket">
+      <origin xyz="0 0 0" rpy="0 0 0" />
+      <geometry>
+        <mesh filename="package://openeta_rm75_v_description/meshes/camera_rolink.STL"
+              scale="1 1 1" />
+      </geometry>
+      <material name="wrist_camera_aluminium"><color rgba="0.75294 0.75294 0.75294 1" /></material>
+    </visual>
+    <collision name="wrist_camera_vendor_bracket_collision">
+      <origin xyz="0 0 0" rpy="0 0 0" />
+      <geometry>
+        <mesh filename="package://openeta_rm75_v_description/meshes/camera_rolink.STL"
+              scale="1 1 1" />
+      </geometry>
+    </collision>
+  </link>
+  <joint name="wrist_camera_bracket_joint" type="fixed">
+    <!-- Use the manufacturer's terminal -X camera shoe.  Pitch the original
+         arm 25 degrees toward the tool tip and seat it 20 mm proximally on
+         the wrist.  The latter preserves a swept keep-out around the 220 mm
+         grasped-part envelope (part radius + exact housing radius + settling
+         clearance), instead of letting a released part tip into the camera.
+         The longer working distance also reduces fixed gripper occlusion. -->
+    <origin xyz="-0.0335 0.0085 -0.07388"
+            rpy="-1.57079632679 -1.1344640138 0" />
+    <parent link="link_7" />
+    <child link="wrist_camera_bracket_link" />
+  </joint>
+  <link name="wrist_camera_housing_link">
+    <inertial>
+      <origin xyz="-0.009 0 -0.011436" rpy="0 0 0" />
+      <mass value="0.03915" />
+      <inertia ixx="7.2029E-06" ixy="0" ixz="0"
+               iyy="7.199E-06" iyz="0" izz="1.1014E-05" />
+    </inertial>
+    <visual name="wrist_camera_vendor_housing">
+      <origin xyz="0 0 0" rpy="0 0 0" />
+      <geometry>
+        <mesh filename="package://openeta_rm75_v_description/meshes/camera_link.STL" />
+      </geometry>
+      <material name="wrist_camera_housing"><color rgba="0.12 0.14 0.16 1" /></material>
+    </visual>
+    <visual name="wrist_camera_rubber_isolator">
+      <origin xyz="-0.009 0 0.0015" rpy="0 0 0" />
+      <geometry><box size="0.034 0.036 0.003" /></geometry>
+      <material name="wrist_camera_rubber"><color rgba="0.035 0.040 0.045 1" /></material>
+    </visual>
+    <visual name="wrist_camera_tilt_hinge">
+      <origin xyz="-0.009 0 0.0045" rpy="1.57079632679 0 0" />
+      <geometry><cylinder radius="0.006" length="0.030" /></geometry>
+      <material name="wrist_camera_hinge"><color rgba="0.32 0.35 0.38 1" /></material>
+    </visual>
+    <visual name="wrist_camera_front_bezel">
+      <origin xyz="-0.009 0 -0.0238" rpy="0 0 0" />
+      <geometry><box size="0.034 0.038 0.0016" /></geometry>
+      <material name="wrist_camera_bezel"><color rgba="0.025 0.030 0.035 1" /></material>
+    </visual>
+    <visual name="wrist_camera_left_depth_lens">
+      <origin xyz="-0.009 -0.012 -0.0250" rpy="0 0 0" />
+      <geometry><cylinder radius="0.0040" length="0.0024" /></geometry>
+      <material name="wrist_camera_depth_glass"><color rgba="0.020 0.090 0.145 0.98" /></material>
+    </visual>
+    <visual name="wrist_camera_rgb_lens">
+      <origin xyz="-0.009 0 -0.0250" rpy="0 0 0" />
+      <geometry><cylinder radius="0.0045" length="0.0024" /></geometry>
+      <material name="wrist_camera_rgb_glass"><color rgba="0.035 0.055 0.075 0.98" /></material>
+    </visual>
+    <visual name="wrist_camera_right_depth_lens">
+      <origin xyz="-0.009 0.012 -0.0250" rpy="0 0 0" />
+      <geometry><cylinder radius="0.0040" length="0.0024" /></geometry>
+      <material name="wrist_camera_depth_glass" />
+    </visual>
+    <visual name="wrist_camera_status_led">
+      <origin xyz="0.006 0.014 -0.0251" rpy="0 0 0" />
+      <geometry><sphere radius="0.0014" /></geometry>
+      <material name="wrist_camera_status_green"><color rgba="0.08 0.72 0.24 1" /></material>
+    </visual>
+    <visual name="wrist_camera_model_badge">
+      <origin xyz="0.005 -0.014 -0.0251" rpy="0 0 0" />
+      <geometry><box size="0.006 0.002 0.0008" /></geometry>
+      <material name="wrist_camera_badge"><color rgba="0.62 0.66 0.70 1" /></material>
+    </visual>
+    <collision name="wrist_camera_vendor_housing_collision">
+      <origin xyz="0 0 0" rpy="0 0 0" />
+      <geometry>
+        <mesh filename="package://openeta_rm75_v_description/meshes/camera_link.STL" />
+      </geometry>
+    </collision>
+  </link>
+  <joint name="wrist_camera_housing_joint" type="fixed">
+    <!-- Seat the camera directly on the original 100.22 mm bracket datum,
+         without another cantilever.  Its optical ray passes outside the
+         Robotiq body and converges on the operation axis 400 mm beyond
+         link_7.  Converging on the 104 mm grasp centre would point straight
+         through the gripper and make fixed self-occlusion unavoidable. -->
+    <origin xyz="0.029031 -0.10022 -0.0005"
+            rpy="-1.55172489 0.06894605 1.40558276" />
+    <parent link="wrist_camera_bracket_link" />
+    <child link="wrist_camera_housing_link" />
   </joint>
   <link name="wrist_camera_optical_frame" />
   <joint name="wrist_camera_optical_joint" type="fixed">
-    <!-- Eye-in-hand RGB-D is centred between the two fingers, immediately
-         beyond the 90 mm Robotiq base.  Gazebo cameras look along local +X;
-         -pi/2 about Y therefore aligns the optical axis with tool +Z. -->
-    <origin xyz="0 0 0.105" rpy="0 -1.57079632679 0" />
-    <parent link="gripper_mount_link" />
+    <!-- The vendor camera mesh occupies local z=[-0.023, 0], with its lens
+         face at -Z.  Gazebo sensors look along +X, so +pi/2 about Y aligns
+         the sensor ray with the physical lens face. -->
+    <origin xyz="0 0 -0.0242" rpy="0 1.57079632679 0" />
+    <parent link="wrist_camera_housing_link" />
     <child link="wrist_camera_optical_frame" />
   </joint>
@@ -565,10 +578,14 @@
     <sensor name="openeta_wrist_rgbd" type="rgbd_camera">
       <camera>
-        <horizontal_fov>1.047</horizontal_fov>
+        <!-- A moderate wide-angle field retains the target after the physical
+             hinge tilt without spending pixels on the near wrist body. -->
+        <horizontal_fov>1.308996938996</horizontal_fov>
         <image><width>640</width><height>480</height><format>R8G8B8</format></image>
         <clip><near>0.02</near><far>5.0</far></clip>
       </camera>
       <always_on>true</always_on>
-      <update_rate>15</update_rate>
+      <!-- Preserve native 640x480 RGB-D quality while avoiding continuous
+           15 Hz eye-in-hand rendering during collision-aware trajectories. -->
+      <update_rate>3</update_rate>
       <topic>openeta_wrist_rgbd</topic>
       <gz_frame_id>wrist_camera_optical_frame</gz_frame_id>

File: extensions/gazebo/assets/robotiq_2f85_vendor/urdf/rm75_robotiq2f85.urdf.xacro (robot description, xacro)
@@ -12,5 +12,9 @@
          simulation-only gap made the Robotiq base visibly float in front of
          the arm and also lengthened every compiled contact pose. -->
-    <joint name="rm75_to_gripper_mount" type="fixed"><parent link="${parent}"/><child link="gripper_mount_link"/><origin xyz="0 0 ${mount_z}"/></joint>
+    <!-- The RM75 camera shoe occupies the terminal -X radial datum.  Rotate
+         the parallel jaws by 90 degrees about the unchanged tool axis so the
+         camera lies in the two-finger symmetry plane instead of behind one
+         finger.  TCP position and approach direction are unchanged. -->
+    <joint name="rm75_to_gripper_mount" type="fixed"><parent link="${parent}"/><child link="gripper_mount_link"/><origin xyz="0 0 ${mount_z}" rpy="0 0 1.57079632679"/></joint>
     <xacro:robotiq_gripper name="robotiq_2f85" prefix="" parent="gripper_mount_link" sim_gazebo="true" include_ros2_control="false"><origin xyz="0 0 0.006"/></xacro:robotiq_gripper>
     <!-- ros2_control is supplied by the repository-local RM75 simulation

File: extensions/gazebo/ros2_ws/src/openeta_rm75_robotiq2f85_sim/urdf/rm75_robotiq2f85_pickplace.urdf.xacro (robot description, xacro)
@@ -7,22 +7,33 @@
   <xacro:rm75_robotiq2f85 parent="link_7" mount_z="0.0"/>
   <xacro:openeta_robotiq_ros2_control controller_config="$(arg controller_config)"/>
-  <xacro:macro name="gz_gripper_position_controller" params="joint topic">
+  <xacro:macro name="gz_gripper_position_controller" params="joint topic p_gain d_gain">
     <gazebo><plugin filename="gz-sim-joint-position-controller-system" name="gz::sim::systems::JointPositionController">
       <joint_name>${joint}</joint_name><topic>${topic}</topic>
-      <p_gain>12.0</p_gain><i_gain>0.0</i_gain><d_gain>0.4</d_gain>
+      <!-- The finger-link inertias range from 1e-5 to 1e-4 kg m^2, and Gazebo updates
+           at 500 Hz.  The former high derivative gain toggled the PID across
+           its target every physics tick, leaving every joint at its 0.5 rad/s
+           velocity limit.  This lower, proportionally damped force loop still
+           rejects gravity error well inside the 0.02 rad action band while
+           allowing a measured stationary terminal state. -->
+      <p_gain>${p_gain}</p_gain><i_gain>0.0</i_gain><d_gain>${d_gain}</d_gain>
       <cmd_max>30.0</cmd_max><cmd_min>-30.0</cmd_min>
     </plugin></gazebo>
   </xacro:macro>
-  <xacro:gz_gripper_position_controller joint="gripper_left_finger_joint" topic="/openeta/gripper/left_outer"/>
-  <xacro:gz_gripper_position_controller joint="gripper_right_finger_joint" topic="/openeta/gripper/right_outer"/>
-  <xacro:gz_gripper_position_controller joint="gripper_left_inner_knuckle_joint" topic="/openeta/gripper/left_inner"/>
-  <xacro:gz_gripper_position_controller joint="gripper_right_inner_knuckle_joint" topic="/openeta/gripper/right_inner"/>
-  <xacro:gz_gripper_position_controller joint="gripper_left_finger_tip_joint" topic="/openeta/gripper/left_tip"/>
-  <xacro:gz_gripper_position_controller joint="gripper_right_finger_tip_joint" topic="/openeta/gripper/right_tip"/>
+  <!-- Outer joints carry the fixed knuckle and finger bodies; the passive
+       inner/tip links have roughly one order of magnitude less effective
+       inertia and therefore use proportionally lower force-loop gains. -->
+  <xacro:gz_gripper_position_controller joint="gripper_left_finger_joint" topic="/openeta/gripper/left_outer" p_gain="4.0" d_gain="0.04"/>
+  <xacro:gz_gripper_position_controller joint="gripper_right_finger_joint" topic="/openeta/gripper/right_outer" p_gain="4.0" d_gain="0.04"/>
+  <xacro:gz_gripper_position_controller joint="gripper_left_inner_knuckle_joint" topic="/openeta/gripper/left_inner" p_gain="0.5" d_gain="0.005"/>
+  <xacro:gz_gripper_position_controller joint="gripper_right_inner_knuckle_joint" topic="/openeta/gripper/right_inner" p_gain="0.5" d_gain="0.005"/>
+  <xacro:gz_gripper_position_controller joint="gripper_left_finger_tip_joint" topic="/openeta/gripper/left_tip" p_gain="0.5" d_gain="0.005"/>
+  <xacro:gz_gripper_position_controller joint="gripper_right_finger_tip_joint" topic="/openeta/gripper/right_tip" p_gain="0.5" d_gain="0.005"/>
   <!-- These are the only grasp-admission inputs: native Gazebo contact data
        from the real vendor fingertip collision meshes. -->
   <gazebo reference="robotiq_85_left_finger_tip_link">
     <sensor name="openeta_native_grasp_left_pad_contact" type="contact">
-      <always_on>true</always_on><update_rate>1000</update_rate>
+      <!-- 250 Hz retains 25 samples in the 100 ms bilateral proof window,
+           far above the three-sample gate, without saturating the bridge. -->
+      <always_on>true</always_on><update_rate>250</update_rate>
       <topic>/openeta/native_grasp/contacts/left_pad</topic>
       <contact><collision>robotiq_85_left_finger_tip_link_collision</collision></contact>
@@ -31,5 +42,5 @@
   <gazebo reference="robotiq_85_right_finger_tip_link">
     <sensor name="openeta_native_grasp_right_pad_contact" type="contact">
-      <always_on>true</always_on><update_rate>1000</update_rate>
+      <always_on>true</always_on><update_rate>250</update_rate>
       <topic>/openeta/native_grasp/contacts/right_pad</topic>
       <contact><collision>robotiq_85_right_finger_tip_link_collision</collision></contact>

File: extensions/gazebo/ros2_ws/src/openeta_rm75_robotiq2f85_sim/urdf/ros2_control.xacro (robot description, xacro)
@@ -31,4 +31,8 @@
               name="gz_ros2_control::GazeboSimROS2ControlPlugin">
         <parameters>${controller_config}</parameters>
+        <!-- Keep the simulated joint inside the trajectory tolerance under
+             load. 0.75 remains below gz_ros2_control's non-overshooting gain
+             of 1.0 while correcting more of each 2 ms position error. -->
+        <position_proportional_gain>0.75</position_proportional_gain>
       </plugin>
     </gazebo>
