Commit message: fix: center wrist RGB-D and flush gripper mount

File: extensions/gazebo/assets/rm75_6fb_v_vendor/urdf/rm75_6fb_v.urdf.xacro (robot description, xacro)
@@ -555,6 +555,9 @@
   <link name="wrist_camera_optical_frame" />
   <joint name="wrist_camera_optical_joint" type="fixed">
-    <origin xyz="0 0 -0.011" rpy="0 1.57079632679 0" />
-    <parent link="camera_link" />
+    <!-- Eye-in-hand RGB-D is centred between the two fingers, immediately
+         beyond the 90 mm Robotiq base.  Gazebo cameras look along local +X;
+         -pi/2 about Y therefore aligns the optical axis with tool +Z. -->
+    <origin xyz="0 0 0.105" rpy="0 -1.57079632679 0" />
+    <parent link="gripper_mount_link" />
     <child link="wrist_camera_optical_frame" />
   </joint>
@@ -564,5 +567,5 @@
         <horizontal_fov>1.047</horizontal_fov>
         <image><width>640</width><height>480</height><format>R8G8B8</format></image>
-        <clip><near>0.05</near><far>5.0</far></clip>
+        <clip><near>0.02</near><far>5.0</far></clip>
       </camera>
       <always_on>true</always_on>

File: extensions/gazebo/assets/robotiq_2f85_vendor/urdf/rm75_robotiq2f85.urdf.xacro (robot description, xacro)
@@ -4,10 +4,13 @@
   <xacro:include filename="$(find openeta_rm75_robotiq2f85_sim)/vendor/robotiq/robotiq_2f_85_macro.urdf.xacro"/>
   <xacro:include filename="$(find openeta_rm75_robotiq2f85_sim)/vendor/robotiq/2f_85.ros2_control.xacro"/>
-  <xacro:macro name="rm75_robotiq2f85" params="parent:=link_7">
+  <xacro:macro name="rm75_robotiq2f85" params="parent:=link_7 mount_z:=0.0">
     <link name="gripper_mount_link">
       <inertial><mass value="0.12"/><inertia ixx="0.00002" iyy="0.00002" izz="0.00002" ixy="0" ixz="0" iyz="0"/></inertial>
       <collision><origin xyz="0 0 0.006"/><geometry><box size="0.08 0.08 0.012"/></geometry></collision>
     </link>
-    <joint name="rm75_to_gripper_mount" type="fixed"><parent link="${parent}"/><child link="gripper_mount_link"/><origin xyz="0 0 0.025"/></joint>
+    <!-- The RM75 terminal mesh ends at its z=0 flange.  The previous 25 mm
+         simulation-only gap made the Robotiq base visibly float in front of
+         the arm and also lengthened every compiled contact pose. -->
+    <joint name="rm75_to_gripper_mount" type="fixed"><parent link="${parent}"/><child link="gripper_mount_link"/><origin xyz="0 0 ${mount_z}"/></joint>
     <xacro:robotiq_gripper name="robotiq_2f85" prefix="" parent="gripper_mount_link" sim_gazebo="true" include_ros2_control="false"><origin xyz="0 0 0.006"/></xacro:robotiq_gripper>
     <!-- ros2_control is supplied by the repository-local RM75 simulation

File: extensions/gazebo/ros2_ws/src/openeta_rm75_robotiq2f85_sim/urdf/rm75_robotiq2f85.urdf.xacro (robot description, xacro)
@@ -5,5 +5,5 @@
   <xacro:include filename="$(find openeta_rm75_robotiq2f85_sim)/vendor/robotiq/rm75_robotiq2f85.urdf.xacro"/>
   <xacro:include filename="$(find openeta_rm75_robotiq2f85_sim)/urdf/ros2_control.xacro"/>
-  <xacro:rm75_robotiq2f85 parent="link_7"/>
+  <xacro:rm75_robotiq2f85 parent="link_7" mount_z="0.0"/>
   <xacro:openeta_robotiq_ros2_control controller_config="$(arg controller_config)"/>
   <xacro:macro name="gz_gripper_position_controller" params="joint topic">

File: extensions/gazebo/ros2_ws/src/openeta_rm75_robotiq2f85_sim/urdf/rm75_robotiq2f85_pickplace.urdf.xacro (robot description, xacro)
@@ -5,5 +5,5 @@
   <xacro:include filename="$(find openeta_rm75_robotiq2f85_sim)/vendor/robotiq/rm75_robotiq2f85.urdf.xacro"/>
   <xacro:include filename="$(find openeta_rm75_robotiq2f85_sim)/urdf/ros2_control.xacro"/>
-  <xacro:rm75_robotiq2f85 parent="link_7"/>
+  <xacro:rm75_robotiq2f85 parent="link_7" mount_z="0.0"/>
   <xacro:openeta_robotiq_ros2_control controller_config="$(arg controller_config)"/>
   <xacro:macro name="gz_gripper_position_controller" params="joint topic">

Commit message: fix(gazebo): align arm mount with pick-place workspace

File: extensions/gazebo/assets/rm75_6fb_v_vendor/urdf/rm75_6fb_v.urdf.xacro (robot description, xacro)
@@ -5,9 +5,14 @@
 <robot
   name="openeta_rm75_v_description">
+  <!-- base_link is the workcell datum shared by Gazebo, MoveIt, cameras, and
+       generated model poses.  The physical pedestal is mounted 200 mm along
+       table X so the near picking area and the receptacle area lie in the
+       same constrained-orientation workspace.  Keep the pedestal inertial,
+       visual, collision, and first joint at this one rigid mounting datum. -->
   <link
     name="base_link">
     <inertial>
       <origin
-        xyz="0.00049987 5.2709E-05 0.060019"
+        xyz="0.20049987 5.2709E-05 0.060019"
         rpy="0 0 0" />
       <mass
@@ -23,5 +28,5 @@
     <visual>
       <origin
-        xyz="0 0 0"
+        xyz="0.20 0 0"
         rpy="0 0 0" />
       <geometry>
@@ -37,5 +42,5 @@
     <collision>
       <origin
-        xyz="0 0 0"
+        xyz="0.20 0 0"
         rpy="0 0 0" />
       <geometry>
@@ -88,10 +93,9 @@
     name="joint_1"
     type="revolute">
-    <!-- Workcell mounting transform: the RM75 pedestal faces away from the
-         work table.  Keep this rotation inside the kinematic tree (rather
-         than applying a Gazebo-only spawn yaw) so TF, MoveIt, IK, collision
-         checking, and the rendered robot all share the same base frame. -->
-    <origin
-      xyz="0 0 0.2405"
+    <!-- Keep the complete workcell mounting transform inside the kinematic
+         tree (rather than applying a Gazebo-only model pose) so TF, MoveIt,
+         IK, collision checking, and the rendered robot remain identical. -->
+    <origin
+      xyz="0.20 0 0.2405"
       rpy="0 0 3.14159265359" />
     <parent
