Commit message: fix: align grasp qualification with four-bar linkage

File: extensions/gazebo/assets/robotiq_2f85_vendor/urdf/rm75_robotiq2f85.urdf.xacro (robot description, xacro)
@@ -4,5 +4,5 @@
   <xacro:include filename="$(find openeta_rm75_robotiq2f85_sim)/vendor/robotiq/robotiq_2f_85_macro.urdf.xacro"/>
   <xacro:include filename="$(find openeta_rm75_robotiq2f85_sim)/vendor/robotiq/2f_85.ros2_control.xacro"/>
-  <xacro:macro name="rm75_robotiq2f85" params="parent:=link_7 mount_z:=0.0">
+  <xacro:macro name="rm75_robotiq2f85" params="parent:=link_7 mount_z:=0.0 exact_four_bar:=false">
     <link name="gripper_mount_link">
       <inertial><mass value="0.12"/><inertia ixx="0.00002" iyy="0.00002" izz="0.00002" ixy="0" ixz="0" iyz="0"/></inertial>
@@ -17,5 +17,5 @@
          finger.  TCP position and approach direction are unchanged. -->
     <joint name="rm75_to_gripper_mount" type="fixed"><parent link="${parent}"/><child link="gripper_mount_link"/><origin xyz="0 0 ${mount_z}" rpy="0 0 1.57079632679"/></joint>
-    <xacro:robotiq_gripper name="robotiq_2f85" prefix="" parent="gripper_mount_link" sim_gazebo="true" include_ros2_control="false"><origin xyz="0 0 0.006"/></xacro:robotiq_gripper>
+    <xacro:robotiq_gripper name="robotiq_2f85" prefix="" parent="gripper_mount_link" sim_gazebo="true" include_ros2_control="false" kinematic_mimic="${not exact_four_bar}"><origin xyz="0 0 0.006"/></xacro:robotiq_gripper>
     <!-- ros2_control is supplied by the repository-local RM75 simulation
          adapter so the arm and gripper share one Gazebo hardware system. -->

File: extensions/gazebo/assets/robotiq_2f85_vendor/urdf/robotiq_2f_85_macro.urdf.xacro (robot description, xacro)
@@ -18,5 +18,6 @@
         gripper_max_speed:=0.150
         gripper_max_force:=235.0
-        gripper_closed_position:=0.7929">
+        gripper_closed_position:=0.7929
+        kinematic_mimic:=true">
         <!-- ros2 control include -->
         <xacro:include filename="$(find openeta_rm75_robotiq2f85_sim)/vendor/robotiq/2f_85.ros2_control.xacro" />
@@ -245,5 +246,7 @@
             <origin xyz="-0.03060114 0.0 0.05490452" rpy="0 0 0" />
             <limit lower="-0.8" upper="0.0" velocity="0.5" effort="50" />
-            <mimic joint="${prefix}gripper_left_finger_joint" multiplier="-1" />
+            <xacro:if value="${kinematic_mimic}">
+                <mimic joint="${prefix}gripper_left_finger_joint" multiplier="-1" />
+            </xacro:if>
         </joint>
         <joint name="${prefix}robotiq_85_left_finger_joint" type="fixed">
@@ -262,5 +265,7 @@
             <axis xyz="0 -1 0" />
             <origin xyz="0.0127 0.0 0.06142" rpy="0 0 0" />
-            <mimic joint="${prefix}gripper_left_finger_joint" />
+            <xacro:if value="${kinematic_mimic}">
+                <mimic joint="${prefix}gripper_left_finger_joint" />
+            </xacro:if>
             <limit lower="0.0" upper="0.8" velocity="0.5" effort="50" />
         </joint>
@@ -270,5 +275,7 @@
             <axis xyz="0 -1 0" />
             <origin xyz="-0.0127 0.0 0.06142" rpy="0 0 0" />
-            <mimic joint="${prefix}gripper_left_finger_joint" multiplier="-1" />
+            <xacro:if value="${kinematic_mimic}">
+                <mimic joint="${prefix}gripper_left_finger_joint" multiplier="-1" />
+            </xacro:if>
             <limit lower="-0.8" upper="0.0" velocity="0.5" effort="50" />
         </joint>
@@ -278,5 +285,7 @@
             <axis xyz="0 -1 0" />
             <origin xyz="0.00563134 0.0 0.04718515" rpy="0 0 0" />
-            <mimic joint="${prefix}gripper_left_finger_joint" multiplier="-1" />
+            <xacro:if value="${kinematic_mimic}">
+                <mimic joint="${prefix}gripper_left_finger_joint" multiplier="-1" />
+            </xacro:if>
             <limit lower="-0.8" upper="0.0" velocity="0.5" effort="50" />
         </joint>
@@ -286,5 +295,7 @@
             <axis xyz="0 -1 0" />
             <origin xyz="-0.00563134 0.0 0.04718515" rpy="0 0 0" />
-            <mimic joint="${prefix}gripper_left_finger_joint" />
+            <xacro:if value="${kinematic_mimic}">
+                <mimic joint="${prefix}gripper_left_finger_joint" />
+            </xacro:if>
             <limit lower="0.0" upper="0.8" velocity="0.5" effort="50" />
         </joint>

File: extensions/gazebo/ros2_ws/src/openeta_rm75_robotiq2f85_sim/urdf/rm75_robotiq2f85_pickplace.urdf.xacro (robot description, xacro)
@@ -5,5 +5,9 @@
   <xacro:include filename="$(find openeta_rm75_robotiq2f85_sim)/vendor/robotiq/rm75_robotiq2f85.urdf.xacro"/>
   <xacro:include filename="$(find openeta_rm75_robotiq2f85_sim)/urdf/ros2_control.xacro"/>
-  <xacro:rm75_robotiq2f85 parent="link_7" mount_z="0.0"/>
+  <!-- Collision qualification uses the same exact four-bar configuration
+       commanded by the native Gazebo adapter, not the vendor's linear mimic
+       approximation.  The arm group remains unchanged; only passive hand
+       joints become explicit RobotState inputs. -->
+  <xacro:rm75_robotiq2f85 parent="link_7" mount_z="0.0" exact_four_bar="true"/>
   <xacro:openeta_robotiq_ros2_control controller_config="$(arg controller_config)"/>
   <xacro:macro name="gz_gripper_position_controller" params="joint topic p_gain d_gain">
